File: demo.kicad_pcb (KiCad board)
At the start: 50 x 30 mm, 3 parts

Commit message: chore: tidy the layout and refresh the BOM
Routine housekeeping ahead of the next build.
Parts:
- removed R2: , Resistor_SMD:R_0603
- added R1: , Resistor_SMD:R_0603, F.Cu at (10.0, 5.00)
Other:
- outline, holes or cut-outs redrawn
Changed lines of the file:
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@@
 (kicad_pcb
   (version 20250114)
-  (title_block (rev "1.0.0"))
-  (gr_rect (start 0 0) (end 50 30) (layer "Edge.Cuts"))
+  (gr_line (start 0 0) (end 50 0) (layer "Edge.Cuts"))
+  (gr_line (start 50 0) (end 50 30) (layer "Edge.Cuts"))
   (footprint "Resistor_SMD:R_0603" (layer "F.Cu") (at 5 5) (property "Reference" "R1"))
-  (footprint "Resistor_SMD:R_0603" (layer "F.Cu") (at 10 5) (property "Reference" "R2"))
+  (footprint "Resistor_SMD:R_0603" (layer "F.Cu") (at 10 5) (property "Reference" "R1"))
   (footprint "Capacitor_SMD:C_0603" (layer "F.Cu") (at 15 5) (property "Reference" "C1"))
 )
